Commit message: updated

File: src/robot_description/urdf/gazebo_control.xacro (robot description, xacro)
@@ -13,5 +13,5 @@
         <!-- output-->
         <odometry_frame>odom</odometry_frame>
-        <robot_base_frame>base_footprint</robot_base_frame>
+        <robot_base_frame>base_link</robot_base_frame>
         <publish_odom>true</publish_odom>
         <publish_odom_tf>true</publish_odom_tf>

File: src/robot_description/urdf/robot.urdf.xacro (robot description, xacro)
@@ -1,5 +1,6 @@
 <?xml version="1.0"?>
 <robot xmlns:xacro="http://www.ros.org/wiki/xacro" name="my_robot">
-  <xacro:include filename="gazebo_control.xacro"/>
+  <!-- <xacro:include filename="gazebo_control.xacro"/> -->
+   <xacro:include filename="ros2_control.xacro" />
   <!-- Definire parametri -->
   <xacro:property name="robot_length" value="0.7"/>
@@ -187,5 +188,5 @@
      <sensor name="laser" type="ray">
         <pose> 0 0 0 0 0 0 </pose>
-        <visualize>true</visualize>
+        <visualize>false</visualize>
         <update_rate>10</update_rate>
         <ray>
@@ -211,3 +212,52 @@
      </sensor>
     </gazebo>
+<!-- Camera principală -->
+<link name="camera_link">
+    <visual>
+      <origin xyz="0 0 0" rpy="0 0 0"/>
+      <geometry>
+        <box size="0.1 0.15 0.15"/>
+      </geometry>
+      <material name="black">
+        <color rgba="0 0 0 1"/>
+      </material>
+    </visual>
+</link>
+<!-- Conectează camera de șasiu -->
+<joint name="base_to_camera" type="fixed">
+    <parent link="base_chassis"/>
+    <child link="camera_link"/>
+    <origin xyz="${robot_length / 2 + 0.05} 0 ${robot_height/2}" rpy="0 0 0"/>
+</joint>
+<!-- Camera optical link -->
+<link name="camera_link_optical"/>
+<!-- Joint pentru camera optică -->
+<joint name="camera_optical_joint" type="fixed">
+    <parent link="camera_link"/>
+    <child link="camera_link_optical"/>
+    <origin xyz="0 0 0" rpy="${-pi/2} 0 ${-pi/2}"/>
+</joint>
+  <gazebo reference="camera_link">
+    <material>Gazebo/Black</material>
+     <sensor name="camera" type="camera">
+        <pose> 0 0 0 0 0 0 </pose>
+        <visualize>true</visualize>
+        <update_rate>10</update_rate>
+        <camera>
+          <horizontal_fov>1.33</horizontal_fov>
+          <image>
+              <format>R8G8B8</format>
+              <width>680</width>
+              <height>480</height>
+          </image>
+            <clip>
+              <near>0.05</near>
+              <far>8.0</far>
+            </clip>
+        </camera>
+        <plugin name="camera_controller" filename="libgazebo_ros_camera.so">
+          <frame_name>camera_link_optical</frame_name>
+        </plugin>
+      </sensor>
+    </gazebo>
 </robot>
